Commit message: new calibrated urdf, updated urdf comments

File: urdf/camera_rig_calibrated.urdf (robot description, URDF)
Before this commit: robot camera_rig, 4 links, 3 joints
Joints:
- removed joint lidar_to_camera
- added joint camera_to_lidar: type fixed, parent camera, child lidar_frame, origin xyz=-0.005000 -0.099000 0.032269 rpy=1.978398 -1.521952 -0.399680
- joint camera_lidar_rig_to_camera: origin xyz=0.027671 0.0 -0.110894 rpy=-1.57 0.0102 -1.57 -> xyz=0.027671 0.0 -0.110894 rpy=-1.570796 0.0102 -1.570796

File: urdf/camera_rig_ideal.urdf (robot description, URDF)
Before this commit: robot camera_rig, 4 links, 3 joints
Joints:
- removed joint lidar_to_camera
- added joint camera_to_lidar: type fixed, parent camera, child lidar_frame, origin xyz= 0.0 -0.099000 0.032269 rpy=1.570796 -1.570796 0.0
- joint camera_lidar_rig_to_camera: origin xyz=0.027671 0.0 -0.110894 rpy=-1.57 0.0102 -1.57 -> xyz=0.027671 0.0 -0.110894 rpy=-1.570796 0.0102 -1.570796

Commit message: fixed rotation transforms

File: urdf/camera_rig_calibrated.urdf (robot description, URDF)
Before this commit: robot camera_rig, 4 links, 3 joints
Joints:
- joint camera_to_lidar: origin xyz=-0.005000 -0.099000 0.032269 rpy=1.978398 -1.521952 -0.399680 -> xyz=-0.004585 -0.097881 0.035223 rpy=-1.167591 -1.523330 2.729625

File: urdf/camera_rig_ideal.urdf (robot description, URDF)
Before this commit: robot camera_rig, 4 links, 3 joints
Joints:
- joint camera_to_lidar: origin xyz= 0.0 -0.099000 0.032269 rpy=1.570796 -1.570796 0.0 -> xyz=-0.004585 -0.097881 0.035223 rpy=-1.167591 -1.523330 2.729625
